File: 2SK3557_LNA_kicad/2SK3557_LNA_kicad.kicad_sch (KiCad schematic)
At the start: 12 parts, among them Q1 BF862

Commit message: add all changes
Parts:
- removed Ci1, Co1: 10n, symbol Device:C
- removed Cs1: 10u, symbol Device:C
- removed Q1: BF862, Package_TO_SOT_THT:TO-92, symbol Transistor_FET:2N3819
- removed Rc1: 500, symbol Device:R
- removed Rl1: 10k, symbol Device:R
- removed Rs1: 80, symbol Device:R
- removed Rs2: 20, symbol Device:R
- removed V3: VSIN, symbol Simulation_SPICE:VSIN
- added C1, C2, C3: 100n, symbol Device:C
- added Q1: 2SK3557, symbol Simulation_SPICE:NJFET
- added R1: 750, symbol Device:R
- added R2: 9k, symbol Device:R
- added R3: 20, symbol Device:R
- added R4: 80, symbol Device:R
- added V2: VSIN, symbol Simulation_SPICE:VSIN
- R5: value 9k -> 330
- R6: value 750 -> 10k
Connections:
- net +5V: now also R2.1
- net GND: now also C1.2, R1.2, R3.2, V2.2
- net Vin: now also C2.1, V2.1
- net Vout: now also R6.1, C3.2
- net at R5.2: now also C3.1, Q1.1 (D); no longer R6.1
- new net: C1.1, R3.1, R4.2
- new net: C2.2, Q1.2 (G), R1.1, R2.2
- new net: Q1.3 (S), R4.1

Commit message: optimize LNA
Parts:
- R1: value 750 -> 1.21k
- R2: value 9k -> 8.87k
- R3: value 20 -> 124
- R4: value 80 -> 124
- R5: value 330 -> 499
Changed lines of the file:
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@@
+	(wire
+		(pts
+			(xy 154.94 101.6) (xy 154.94 102.87)
+		)
+		(stroke
+			(width 0)
+			(type default)
+		)
+	)
 	(wire
 		(pts
@@
 		(pts
 			(xy 130.81 96.52) (xy 137.16 96.52)
-		)
-		(stroke
-			(width 0)
-			(type default)
-		)
-	)
-	(wire
-		(pts
-			(xy 154.94 101.6) (xy 154.94 102.87)
 		)
 		(stroke
@@
 			)
 		)
-		(property "Value" "9k"
+		(property "Value" "8.87k"
 			(at 139.7 88.8999 0)
 			(effects
@@
 			)
 		)
-		(property "Value" "20"
+		(property "Value" "124"
 			(at 157.48 116.8399 0)
 			(effects
@@
 			)
 		)
-		(property "Value" "750"
+		(property "Value" "1.21k"
 			(at 139.7 105.4099 0)
 			(effects
@@
 			)
 		)
-		(property "Value" "330"
+		(property "Value" "499"
 			(at 157.48 86.3599 0)
 			(effects
@@
 			)
 		)
-		(property "Value" "80"
+		(property "Value" "124"
 			(at 157.48 107.9499 0)
 			(effects

Commit message: new vals
Parts:
- R1: value 1.21k -> 30k
- R2: value 8.87k -> 100k
- R3: value 124 -> 27
- R4: value 124 -> 75
- R5: value 499 -> 200
Connections:
- net GND: now also R4.2; no longer R3.2
- net at R4.1: now also C1.1, R3.2; no longer Q1.3 (S)
- new net: Q1.3 (S), R3.1
Other:
- moved on the sheet: C1, R3, R4, R6
Changed lines of the file:
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@@
 	(paper "A4")
-	(junction
-		(at 154.94 111.76)
-		(diameter 0)
-		(color 0 0 0 0)
-	)
 	(junction
 		(at 137.16 96.52)
@@
 	)
 	(junction
-		(at 158.75 119.38)
+		(at 154.94 113.03)
 		(diameter 0)
 		(color 0 0 0 0)
@@
 		(color 0 0 0 0)
 	)
+	(junction
+		(at 154.94 120.65)
+		(diameter 0)
+		(color 0 0 0 0)
+	)
 	(wire
 		(pts
-			(xy 154.94 119.38) (xy 158.75 119.38)
+			(xy 187.96 93.98) (xy 187.96 91.44)
 		)
 		(stroke
@@
 	(wire
 		(pts
-			(xy 186.69 92.71) (xy 186.69 91.44)
+			(xy 154.94 113.03) (xy 167.64 113.03)
 		)
 		(stroke
@@
 	(wire
 		(pts
-			(xy 154.94 111.76) (xy 163.83 111.76)
+			(xy 154.94 120.65) (xy 154.94 123.19)
 		)
 		(stroke
@@
 	(wire
 		(pts
-			(xy 158.75 119.38) (xy 163.83 119.38)
+			(xy 154.94 120.65) (xy 167.64 120.65)
 		)
 		(stroke
@@
 	(wire
 		(pts
-			(xy 154.94 110.49) (xy 154.94 111.76)
+			(xy 154.94 110.49) (xy 154.94 113.03)
 		)
 		(stroke
@@
 	(wire
 		(pts
-			(xy 154.94 101.6) (xy 154.94 102.87)
+			(xy 176.53 91.44) (xy 187.96 91.44)
 		)
 		(stroke
@@
 	(wire
 		(pts
-			(xy 176.53 91.44) (xy 186.69 91.44)
+			(xy 130.81 96.52) (xy 137.16 96.52)
 		)
 		(stroke
@@
 	(wire
 		(pts
-			(xy 130.81 96.52) (xy 137.16 96.52)
+			(xy 154.94 101.6) (xy 154.94 102.87)
 		)
 		(stroke
@@
 	)
 	(label "Vout"
-		(at 186.69 91.44 0)
+		(at 187.96 91.44 0)
 		(effects
 			(font
@@
 	(symbol
 		(lib_id "Device:C")
-		(at 163.83 115.57 0)
+		(at 167.64 116.84 0)
 		(unit 1)
 		(exclude_from_sim no)
@@
 		(fields_autoplaced yes)
 		(property "Reference" "C1"
-			(at 167.64 114.2999 0)
+			(at 171.45 115.5699 0)
 			(effects
 				(font
@@
 		)
 		(property "Value" "100n"
-			(at 167.64 116.8399 0)
-			(effects
-				(font
-					(size 1.27 1.27)
-				)
-				(justify left)
-			)
-		)
-		(property "Footprint" ""
-			(at 164.7952 119.38 0)
+			(at 171.45 118.1099 0)
+			(effects
+				(font
+					(size 1.27 1.27)
+				)
+				(justify left)
+			)
+		)
+		(property "Footprint" ""
+			(at 168.6052 120.65 0)
 			(effects
 				(font
@@
 		)
 		(property "Datasheet" "~"
-			(at 163.83 115.57 0)
+			(at 167.64 116.84 0)
 			(effects
 				(font
@@
 		)
 		(property "Description" "Unpolarized capacitor"
-			(at 163.83 115.57 0)
+			(at 167.64 116.84 0)
 			(effects
 				(font
@@
 	(symbol
 		(lib_id "Device:R")
-		(at 186.69 96.52 0)
+		(at 187.96 97.79 0)
 		(unit 1)
 		(exclude_from_sim no)
@@
 		(fields_autoplaced yes)
 		(property "Reference" "R6"
-			(at 189.23 95.2499 0)
+			(at 190.5 96.5199 0)
 			(effects
 				(font
@@
 		)
 		(property "Value" "10k"
-			(at 189.23 97.7899 0)
-			(effects
-				(font
-					(size 1.27 1.27)
-				)
-				(justify left)
-			)
-		)
-		(property "Footprint" ""
-			(at 184.912 96.52 90)
+			(at 190.5 99.0599 0)
+			(effects
+				(font
+					(size 1.27 1.27)
+				)
+				(justify left)
+			)
+		)
+		(property "Footprint" ""
+			(at 186.182 97.79 90)
 			(effects
 				(font
@@
 		)
 		(property "Datasheet" "~"
-			(at 186.69 96.52 0)
+			(at 187.96 97.79 0)
 			(effects
 				(font
@@
 		)
 		(property "Description" "Resistor"
-			(at 186.69 96.52 0)
+			(at 187.96 97.79 0)
 			(effects
 				(font
@@
 			)
 		)
-		(property "Value" "8.87k"
+		(property "Value" "100k"
 			(at 139.7 88.8999 0)
 			(effects
@@
 	(symbol
 		(lib_id "Device:R")
-		(at 154.94 115.57 0)
+		(at 154.94 106.68 0)
 		(unit 1)
 		(exclude_from_sim no)
@@
 		(fields_autoplaced yes)
 		(property "Reference" "R3"
-			(at 157.48 114.2999 0)
-			(effects
-				(font
-					(size 1.27 1.27)
-				)
-				(justify left)
-			)
-		)
-		(property "Value" "124"
-			(at 157.48 116.8399 0)
-			(effects
-				(font
-					(size 1.27 1.27)
-				)
-				(justify left)
-			)
-		)
-		(property "Footprint" ""
-			(at 153.162 115.57 90)
+			(at 157.48 105.4099 0)
+			(effects
+				(font
+					(size 1.27 1.27)
+				)
+				(justify left)
+			)
+		)
+		(property "Value" "27"
+			(at 157.48 107.9499 0)
+			(effects
+				(font
+					(size 1.27 1.27)
+				)
+				(justify left)
+			)
+		)
+		(property "Footprint" ""
+			(at 153.162 106.68 90)
 			(effects
 				(font
@@
 		)
 		(property "Datasheet" "~"
-			(at 154.94 115.57 0)
+			(at 154.94 106.68 0)
 			(effects
 				(font
@@
 		)
 		(property "Description" "Resistor"
-			(at 154.94 115.57 0)
+			(at 154.94 106.68 0)
 			(effects
 				(font
@@
 	(symbol
 		(lib_id "power:GND")
-		(at 158.75 119.38 0)
+		(at 154.94 123.19 0)
 		(unit 1)
 		(exclude_from_sim no)
@@
 		(fields_autoplaced yes)
 		(property "Reference" "#PWR02"
-			(at 158.75 125.73 0)
+			(at 154.94 129.54 0)
 			(effects
 				(font
@@
 		)
 		(property "Value" "GND"
-			(at 158.75 124.46 0)
-			(effects
-				(font
-					(size 1.27 1.27)
-				)
-			)
-		)
-		(property "Footprint" ""
-			(at 158.75 119.38 0)
+			(at 154.94 128.27 0)
+			(effects
+				(font
+					(size 1.27 1.27)
+				)
+			)
+		)
+		(property "Footprint" ""
+			(at 154.94 123.19 0)
 			(effects
 				(font
@@
 		)
 		(property "Datasheet" ""
-			(at 158.75 119.38 0)
+			(at 154.94 123.19 0)
 			(effects
 				(font
@@
 		)
 		(property "Description" "Power symbol creates a global label with name \"GND\" , ground"
-			(at 158.75 119.38 0)
+			(at 154.94 123.19 0)
 			(effects
 				(font
@@
 		(on_board yes)
 		(dnp no)
-		(fields_autoplaced yes)
 		(property "Reference" "R1"
 			(at 139.7 102.8699 0)
@@
 			)
 		)
-		(property "Value" "1.21k"
-			(at 139.7 105.4099 0)
+		(property "Value" "30k"
+			(at 139.7 104.902 0)
 			(effects
 				(font
@@
 	(symbol
 		(lib_id "power:GND")
-		(at 186.69 100.33 0)
+		(at 187.96 101.6 0)
 		(unit 1)
 		(exclude_from_sim no)
@@
 		(fields_autoplaced yes)
 		(property "Reference" "#PWR07"
-			(at 186.69 106.68 0)
+			(at 187.96 107.95 0)
 			(effects
 				(font
@@
 		)
 		(property "Value" "GND"
-			(at 186.69 105.41 0)
-			(effects
-				(font
-					(size 1.27 1.27)
-				)
-			)
-		)
-		(property "Footprint" ""
-			(at 186.69 100.33 0)
+			(at 187.96 106.68 0)
+			(effects
+				(font
+					(size 1.27 1.27)
+				)
+			)
+		)
+		(property "Footprint" ""
+			(at 187.96 101.6 0)
 			(effects
 				(font
@@
 		)
 		(property "Datasheet" ""
-			(at 186.69 100.33 0)
+			(at 187.96 101.6 0)
 			(effects
 				(font
@@
 		)
 		(property "Description" "Power symbol creates a global label with name \"GND\" , ground"
-			(at 186.69 100.33 0)
+			(at 187.96 101.6 0)
 			(effects
 				(font
@@
 			)
 		)
-		(property "Value" "499"
+		(property "Value" "200"
 			(at 157.48 86.3599 0)
 			(effects
@@
 	(symbol
 		(lib_id "Device:R")
-		(at 154.94 106.68 0)
+		(at 154.94 116.84 0)
 		(unit 1)
 		(exclude_from_sim no)
@@
 		(fields_autoplaced yes)
 		(property "Reference" "R4"
-			(at 157.48 105.4099 0)
-			(effects
-				(font
-					(size 1.27 1.27)
-				)
-				(justify left)
-			)
-		)
-		(property "Value" "124"
-			(at 157.48 107.9499 0)
-			(effects
-				(font
-					(size 1.27 1.27)
-				)
-				(justify left)
-			)
-		)
-		(property "Footprint" ""
-			(at 153.162 106.68 90)
+			(at 157.48 115.5699 0)
+			(effects
+				(font
+					(size 1.27 1.27)
+				)
+				(justify left)
+			)
+		)
+		(property "Value" "75"
+			(at 157.48 118.1099 0)
+			(effects
+				(font
+					(size 1.27 1.27)
+				)
+				(justify left)
+			)
+		)
+		(property "Footprint" ""
+			(at 153.162 116.84 90)
 			(effects
 				(font
@@
 		)
 		(property "Datasheet" "~"
-			(at 154.94 106.68 0)
+			(at 154.94 116.84 0)
 			(effects
 				(font
@@
 		)
 		(property "Description" "Resistor"
-			(at 154.94 106.68 0)
-			(effects
-				(font
+			(at 154.94 116.84 0)
+			(effects
+				(font
